File: electronics/eagle/incubator.brd (EAGLE design)
At the start: 62.2 x 94.9 mm, 31 parts, among them Q1 IRLZ44N, Q2 IRLZ44N, Q3 IRLZ44N, Q4 IRLZ44N, X1 PI Connector, X2 PWM0, X3 PWM1, X4 GPIO5, X5 GPIO6

Commit message: aaded pcb
Parts:
- removed X1: PI Connector, con-molex:87758-4016
- added JP10: PI Connector, pinhead:2X20
- added JP6: 1W Supply, pinhead:1X03
- added JP7: 1Wire Supply, pinhead:1X02
- added JP8: 3.3v, pinhead:1X02
- added JP9: 5v, pinhead:1X02
- moved Q1 54.0 mm to (44.3, 85.9)
- moved R1 52.4 mm to (45.0, 76.1)
- moved R10 52.4 mm to (23.6, 61.1)
- moved R11 52.4 mm to (24.1, 18.2)
- moved R5 52.4 mm to (44.9, 72.3)
- moved R8 52.4 mm to (44.5, 30.5)
- moved R9 52.4 mm to (23.4, 72.5)
- moved OK1 52.4 mm to (30.4, 73.2)
- moved OK2 52.4 mm to (30.4, 51.6)
- moved OK3 52.4 mm to (29.1, 9.65)
- moved OK4 52.4 mm to (29.2, 30.5)
- moved Q2 52.4 mm to (44.6, 62.7)
- moved Q3 52.4 mm to (44.6, 20.8)
- moved Q4 52.4 mm to (44.5, 41.9)
- moved R12 52.4 mm to (24.1, 39.4)
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Connections:
- removed net GPIO5: R11.1, X1.29
- removed net GPIO6: R12.1, X1.31
- new net 1WIRE_VCC: JP1.1, JP2.1, JP3.1, JP4.1, JP5.1, JP6.2, R13.2
- new net GPIO17: JP10.11, R11.1
- new net GPIO27: JP10.13, R12.1
- new net N$12: JP6.3, JP7.2
- new net VCC5V: JP10.2, JP9.1
- net 1-WIRE: now also JP10.7; no longer X1.7
- net GND: now also JP10.39, JP7.1, JP8.2, JP9.2; no longer X1.39
- net OUT3: now also X4.3; no longer X4.2
- net OUT4: now also X5.3; no longer X5.2
- net PWM0: now also JP10.32; no longer X1.32
- net PWM1: now also JP10.33; no longer X1.33
- net PWMOUT1: now also X2.3; no longer X2.2
- net PWMOUT2: now also X3.3; no longer X3.2
- net SUPPLY1: now also X2.2; no longer X2.3
- net SUPPLY2: now also X3.2; no longer X3.3
- net SUPPLY3: now also X4.2; no longer X4.3
- net SUPPLY4: now also X5.2; no longer X5.3
- net VCC3.3: now also JP10.1, JP6.1, JP8.1; no longer JP1.1, JP2.1, JP3.1, JP4.1, JP5.1, R13.2, X1.1
Routing:
- net GPIO5: track 52.6 -> 0.00 mm
- net GPIO17: track 0.00 -> 33.8 mm
- net GPIO6: track 33.7 -> 0.00 mm
- net 1WIRE_VCC: track 0.00 -> 27.1 mm
- net SUPPLY3: track 13.6 -> 32.4 mm
- net SUPPLY4: track 13.9 -> 32.1 mm
- net SUPPLY2: track 13.5 -> 31.0 mm
- net SUPPLY1: track 14.3 -> 31.9 mm
- net VCC3.3: track 32.3 -> 15.8 mm, vias 1 -> 0
- net GPIO27: track 0.00 -> 15.1 mm
- net GND: track 0.00 -> 11.4 mm
- net PWMOUT1: track 6.63 -> 16.8 mm
- net N$12: track 0.00 -> 9.93 mm
- net OUT4: track 6.77 -> 15.1 mm
- net PWMOUT2: track 6.48 -> 14.8 mm
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- added copper zone on layer 16, net GND0
- added copper zone on layer 16, net GND2
- added copper zone on layer 16, net GND3
- added copper zone on layer 16, net GND4
Other:
- board size 62.2 x 94.9 mm -> 69.8 x 94.9 mm
- board text added: "+"
- board text added: "1"
- board text added: "1-wire"
- board text added: "1w"
- board text added: "3.3"
- board text added: "3.3v"
- board text added: "5v"
- board text added: "AARHUS UNIVERSITY"
- board text added: "Ext"
- board text added: "GND"
- board text added: "GPIO12"
- board text added: "GPIO13"
- board text added: "GPIO17"
- board text added: "GPIO27"
- board text added: "OUT"
- board text added: "PI"
- board text added: "PWM0"
- board text added: "PWM1"
