File: electronics/eagle/incubator.sch (EAGLE design)
At the start: 31 parts, among them Q1 IRLZ44N, Q2 IRLZ44N, Q3 IRLZ44N, Q4 IRLZ44N, X1 87758-4016

Commit message: updated pcb design
Parts:
- JP1: value (none) -> Temp1
- JP2: value (none) -> Temp2
- JP3: value (none) -> Temp3
- JP4: value (none) -> Temp4
- JP5: value (none) -> Temp5
- X1: value 87758-4016 -> PI Connector
- X2: value (none) -> PWM0; device con-wago-500:W237-103 -> con-wago-508:W237-04P
- X3: value (none) -> PWM1; device con-wago-500:W237-103 -> con-wago-508:W237-04P
- X4: value (none) -> GPIO5; device con-wago-500:W237-103 -> con-wago-508:W237-04P
- X5: value (none) -> GPIO6; device con-wago-500:W237-103 -> con-wago-508:W237-04P
Connections:
- removed net VCC: JP1.1, JP2.1, JP3.1, JP4.1, JP5.1, R13.2
- net SUPPLY1: now also X2-4.KL
- net SUPPLY2: now also X3-4.KL
- net SUPPLY3: now also X4-4.KL
- net SUPPLY4: now also X5-4.KL
- net VCC3.3: now also JP1.1, JP2.1, JP3.1, JP4.1, JP5.1, R13.2

Commit message: aaded pcb
Parts:
- removed X1: PI Connector, con-molex:87758-4016
- added JP10: PI Connector, pinhead:PINHD-2X20
- added JP6: 1W Supply, pinhead:PINHD-1X3
- added JP7: 1Wire Supply, pinhead:PINHD-1X2
- added JP8: 3.3v, pinhead:PINHD-1X2
- added JP9: 5v, pinhead:PINHD-1X2
Connections:
- removed net GPIO5: R11.1, X1-29.S
- removed net GPIO6: R12.1, X1-31.S
- new net 1WIRE_VCC: JP1.1, JP2.1, JP3.1, JP4.1, JP5.1, JP6.2, R13.2
- new net GPIO17: JP10.11, R11.1
- new net GPIO27: JP10.13, R12.1
- new net N$12: JP6.3, JP7.2
- new net VCC5V: JP10.2, JP9.1
- net 1-WIRE: now also JP10.7; no longer X1-7.S
- net GND: now also JP10.39, JP7.1, JP8.2, JP9.2; no longer X1-39.S
- net OUT3: now also X4-3.KL; no longer X4-2.KL
- net OUT4: now also X5-3.KL; no longer X5-2.KL
- net PWM0: now also JP10.32; no longer X1-32.S
- net PWM1: now also JP10.33; no longer X1-33.S
- net PWMOUT1: now also X2-3.KL; no longer X2-2.KL
- net PWMOUT2: now also X3-3.KL; no longer X3-2.KL
- net SUPPLY1: now also X2-2.KL; no longer X2-3.KL
- net SUPPLY2: now also X3-2.KL; no longer X3-3.KL
- net SUPPLY3: now also X4-2.KL; no longer X4-3.KL
- net SUPPLY4: now also X5-2.KL; no longer X5-3.KL
- net VCC3.3: now also JP10.1, JP6.1, JP8.1; no longer JP1.1, JP2.1, JP3.1, JP4.1, JP5.1, R13.2, X1-1.S
Other:
- moved on the sheet: X2-2, X2-3, X3-2, X3-3, X4-2, X4-3, X5-2, X5-3
